Commit message: feat: Implement asset generation framework with Builder, Validator, and Exporter patterns
- Added a comprehensive asset generation framework in `asset_generator.py` that includes:
  - Builder classes for different levels (Joint, Finger, Palm, Hand) to construct HandCfg objects.
  - Validator classes to ensure the physical validity of generated assets.
  - Exporter classes for exporting HandCfg objects to URDF and YAML formats.
- Enhanced the URDF file for test assets by adjusting visual and collision properties.
- Updated requirement documentation to address challenges in ensuring physical validity and diversity in generated assets.

File: source/anymani/anymani/assets/custom/tips/test.urdf (robot description, URDF)
Before this commit: robot test, 1 links, 0 joints
Links:
- link base_link: geometry visual box size=0.04 0.04 0.04

Commit message: feat: 添加自定义构建器配置类和基础几何构建器，更新资产生成框架

File: source/anymani/anymani/assets/custom/tips/test.urdf (robot description, URDF)
Before this commit: robot test, 1 links, 0 joints
Links:
- link base_link: geometry collision cylinder length=0.5 radius=0.5; collision sphere radius=0.5
