Commit message: feat: Enhance joint builders and add custom finger tip assets 重要特性，框架基本构建
- Updated `CustomJointBuilder` with additional notes on algorithm customization for different finger mesh origins.
- Introduced `PrimJointBuilderCfg` with a new `axis` attribute for revolute joints.
- Added new STL files for various finger tip designs: `round_finger_tip`, `thinner_finger_tip`, `wedge_finger_tip`, and their soft variants.
- Created URDF files for testing custom finger tips, including a new `test_custom.urdf` for collision geometry.
- Updated `requirement.md` to reflect new insights and considerations for joint builders.
- Added a comprehensive research background document outlining the goals and methodologies for in-hand manipulation framework development.

File: source/anymani/anymani/assets/custom/tips/test _custom.urdf (robot description, URDF)
Before this commit: robot test, 2 links, 1 joints
Links:
- removed link tip
- link base_link: geometry collision cylinder length=0.5 radius=0.5; collision sphere radius=0.5
Joints:
- removed joint tip_joint
