Commit message: feat: Enhance custom joint and tip builders with new configuration options
- Updated `CustomJointBuilderCfg` to include `mesh_offset` for flexible mesh positioning and added internal parsing for `_mesh_offset_6d`.
- Introduced `CustomTipBuilderCfg` for specific configurations related to fingertip construction, including scale and tip type.
- Refined `PrimJointBuilderCfg` to clarify the handling of the `origin` field and its relevance in joint construction.
- Added new URDF files for thumb and fingertip configurations, including detailed collision geometries and inertial properties.
- Introduced new STL files for fingertip designs and updated documentation to reflect changes in the joint building process.
- Enhanced requirement documentation to address physical realism and mesh feature extraction considerations.

File: source/anymani/anymani/assets/custom/tips/test_leap_cube.urdf (robot description, URDF)
Before this commit: robot test, 2 links, 1 joints
Links:
- link tip: geometry collision mesh filename=/home/hac/isaac/AnyMani/source/anymani/anymani/assets/custo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 scale=0.001 0.001 0.001; visual mesh filename=/home/hac/isaac/AnyMani/source/anymani/anymani/assets/custo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 scale=0.001 0.001 0.001
