Commit message: feat(assets): add post-mutate restore and quick entrypoints

File: source/anymani/anymani/assets/custom/tips/test_leap_origin.urdf (robot description, URDF)
Before this commit: robot test, 2 links, 1 joints
Links:
- link tip: geometry collision mesh filename=finger_tip_soft.stl scale=0.001 0.001 0.001; visual mesh filename=finger_tip_soft.stl scale=0.001 0.001 0.001

File: source/anymani/anymani/assets/custom/tips/test_wedge.urdf (robot description, URDF)
Before this commit: robot test, 2 links, 1 joints
Links:
- link tip: geometry collision mesh filename=wedge_finger_tip_soft.stl scale=0.0006896551724 0.0006896551724 0.0006896551724; visual mesh filename=wedge_finger_tip_soft.stl scale=0.0006896551724 0.0006896551724 0.0006896551724
